Commit message: finnally rtabmap chalyo main change gareko vaneko inliner haru ho

File: src/CSLAM-UAV/drone_slam_pkg/urdf/base_link.urdf (robot description, URDF)
Before this commit: robot x500_drone, 6 links, 5 joints
Joints:
- joint depth_to_camera: origin (none) -> xyz=0.12 0.03 0.242 rpy=0 0 0

Commit message: problem was with the tf which was creating bad 2d as well as 3d map

File: src/CSLAM-UAV/drone_slam_pkg/urdf/base_link.urdf (robot description, URDF)
Before this commit: robot x500_drone, 6 links, 5 joints
Joints:
- joint depth_to_camera: origin xyz=0.12 0.03 0.242 rpy=0 0 0 -> xyz=0.12 0.03 0.242 rpy=-1.570796327 0 -1.570796327
